File: ch32_v303cb.kicad_pcb (KiCad board)
At the start: 4 copper layers, 33.7 x 20.4 mm, 80 parts, among them J1 Conn_02x05_Odd_Even, J2 Conn_02x05_Odd_Even, J3 Conn_02x08_Odd_Even, J4 Conn_01x02_Socket, J5 Conn_02x05_Odd_Even, J6 Conn_02x05_Odd_Even, SW1 SW_Push, U1 CH32V30xCxTx, U2 AP2112K-3.3TRG1, Y1 Crystal_GND24

Commit message: Renumber components by PCB position; add interactive pinout configurator
Reference designators for all components (connectors, R, C, LED, including
the 10 reused filter-sheet instances) now follow physical placement on the
board instead of arbitrary KiCad placement order. Connectors specifically
go clockwise starting from the programmer header (J1), with the USB header
last (J6). Verified electrically identical: ERC/DRC violation counts match
before/after, and the exported netlist has the exact same 79 nets once old
refs are mapped to new ones.

Also adds docs/ — a self-contained interactive HTML page listing all 5 IDC
headers with GPIO-to-peripheral tables and checkboxes for alternate pin
functions (AFIO remap groups), highlighting pin conflicts live.
Parts:
- renumbered C9 to C1, C13 to C10, C15 to C11, C6 to C12, C1 to C13, C22 to C14, C19 to C15, C2 to C16, C21 to C17, C5 to C18, C17 to C19, C11 to C2, C3 to C20, C20 to C21, C18 to C22, C10 to C3, C7 to C4, C8 to C5, C12 to C6, C16 to C7, C4 to C8, C14 to C9, J5 to J1, J3 to J2, J2 to J3, J1 to J4, J6 to J5, J4 to J6, LED5 to LED1, LED4 to LED2, LED2 to LED4, LED1 to LED5, R36 to R1, R28 to R10, R32 to R11, R15 to R12, R26 to R13, R31 to R14, R30 to R15, R38 to R16, R39 to R17, R22 to R18, R18 to R19, R25 to R2, R34 to R20, R35 to R21, R19 to R22, R6 to R23, R1 to R24, R2 to R25, R33 to R26, R4 to R27, R9 to R28, R3 to R29, R27 to R3, R16 to R30, R13 to R31, R8 to R32, R12 to R33, R7 to R34, R5 to R35, R11 to R36, R10 to R37, R20 to R38, R21 to R39, R29 to R4, R14 to R5, R37 to R6, R17 to R7, R23 to R8, R24 to R9
